File: Kicad/PC-8001_SD.kicad_pcb (KiCad board)
At the start: 2 copper layers, 100 x 100 mm, 20 parts, among them J1 PC-8001 BUS, J2 Micro_SD_Card_Kit, J3 Conn_01x25, U1 74LS04, U2 74LS30, U3 74LS30, U4 8255, U5 2764, U6 Arduino_Pro_Mini_5V

Commit message: Add files via upload
Parts:
- J2: footprint MZ80k_SD:AE-microSD-LLCNV -> Kicad:AE-microSD-LLCNV
- U6: footprint MZ80k_SD:Arduino_Pro_Mini -> Kicad:Arduino_Pro_Mini

Commit message: Add files via upload
Parts:
- added J4: MicroSD Card Adapter, Connector_PinSocket_2.54mm:PinSocket_1x06_P2.54mm_Vertical, F.Cu at (145.5, 97.2)
- added S2: SLIDE SWITCH, Button_Switch_THT:SW_CuK_JS202011CQN_DPDT_Straight, F.Cu at (124.2, 85.5)
- moved C4 8.32 mm to (127.7, 96.4)
- moved U4 8.32 mm to (137.2, 148.5)
- moved C3 7.55 mm to (112.0, 81.0)
- moved U1 7.55 mm to (114.4, 135.4)
- moved C1 7.55 mm to (111.9, 139.2)
- moved U2 7.55 mm to (114.6, 105.8)
- moved U3 7.55 mm to (114.6, 77.5)
- moved C2 7.55 mm to (111.9, 109.5)
- moved U5 2.92 mm to (131.7, 77.5)
- moved C5 2.92 mm to (127.9, 68.2)
Connections:
- net Net-(J2-Pad5) renamed /SCK
- net Net-(J2-Pad6) renamed /MISO
- net Net-(J2-Pad7) renamed /MOSI
- net Net-(J2-Pad8) renamed /CS
- S1 pad 2: /~ROMDS3 -> Net-(S1-Pad2)
- U1 pad 3: /~ROMDS3 -> Net-(S1-Pad2)
- U1 pad 4: Net-(U1-Pad4) -> Net-(S2-Pad4)
- U3 pad 5: Net-(U1-Pad4) -> Net-(S2-Pad5)
Routing:
- net Net-(S1-Pad2): track 0.00 -> 114.4 mm
- net Net-(U1-Pad4): track 67.4 -> 0.00 mm
- net Net-(S2-Pad4): track 0.00 -> 43.9 mm
- net /A5: track 104.4 -> 62.8 mm
- net /~ROMDS3: track 96.2 -> 64.4 mm
- net Net-(S2-Pad5): track 0.00 -> 28.2 mm
- net /A15: track 68.8 -> 47.1 mm
- net GND: track 294.8 -> 314.7 mm, vias 3 -> 1
- net /A10: track 81.6 -> 100.8 mm
- net +5V: track 273.3 -> 290.8 mm
- net Net-(U4-Pad10): track 23.3 -> 40.3 mm
- net Net-(U4-Pad19): track 32.5 -> 48.1 mm
- net /SCK: track 45.2 -> 59.5 mm, vias 1 -> 0
- net Net-(U2-Pad8): track 76.8 -> 62.8 mm, vias 1 -> 2
- net /D5: track 113.6 -> 101.2 mm, vias 0 -> 1
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Other:
- board text added: "EXT"
- board text added: "FIX"
- board text added: "PC-8001_SD Rev1.2"
- board text added: "ROMDS3"
- board text removed: "PC-8001_SD Rev1.1"
