File: Kicad/PC-8001_SD.sch (KiCad schematic (older format))
At the start: 16 parts, among them J1 PC-8001 BUS, J2 Micro_SD_Card_Kit, J3 Conn_01x25, U1 74LS04, U2 74LS30, U3 74LS30, U4 8255, U5 2764, U6 Arduino_Pro_Mini_5V

Commit message: Add files via upload
Parts:
- J2: footprint MZ80k_SD:AE-microSD-LLCNV -> Kicad:AE-microSD-LLCNV
- U6: footprint MZ80k_SD:Arduino_Pro_Mini -> Kicad:Arduino_Pro_Mini
Changed lines of the file:
@@
 F 0 "J2" H 13450 2900 50  0000 L CNN
 F 1 "Micro_SD_Card_Kit" H 13950 2900 50  0000 L CNN
-F 2 "MZ80k_SD:AE-microSD-LLCNV" H 15100 2500 50  0001 C CNN
+F 2 "Kicad:AE-microSD-LLCNV" H 15100 2500 50  0001 C CNN
 F 3 "http://katalog.we-online.de/em/datasheet/693072010801.pdf" H 13950 2200 50  0001 C CNN
 	1    13950 2200
@@
 F 0 "U6" H 12300 5689 60  0000 C CNN
 F 1 "Arduino_Pro_Mini_5V" H 12300 5583 60  0000 C CNN
-F 2 "MZ80k_SD:Arduino_Pro_Mini" H 13100 4050 60  0001 C CNN
+F 2 "Kicad:Arduino_Pro_Mini" H 13100 4050 60  0001 C CNN
 F 3 "https://www.sparkfun.com/products/11113" H 12500 3600 60  0001 C CNN
 	1    12300 4800

Commit message: Add files via upload
Parts:
- added J4: MicroSD Card Adapter, Connector_PinSocket_2.54mm:PinSocket_1x06_P2.54mm_Vertical, symbol Connector_Generic:Conn_01x06
- added S2: SLIDE SWITCH, Button_Switch_THT:SW_CuK_JS202011CQN_DPDT_Straight, symbol Switch:SW_Push_DPDT
Connections:
- net labels added: CS, MISO, MOSI, SCK
- wire segments 286 -> 303
Other:
- moved on the sheet: J1, J3
